File: MAX-M8/MAX-M8_Breakout.brd (EAGLE design)
At the start: 33 x 23.6 mm, 18 parts, among them J1 CONN_92.54_SCREW, J2 U.FL, U1 MAX-M8W

Commit message: Updated MAX-M8 breakout with active antenna support
Parts:
- added C26: 47pF, bschulz_passives:C0402
- added FB7: 30Ω/1.8A, SparkFun-Coils:0603
- added R28: 10, bschulz_passives:R0402
Connections:
- new net ANT_VCC: C26.1, FB7.2, R28.1
- net GND: now also C26.2
- net GPS_ANT: now also FB7.1
- net VCC_RF: now also R28.2
Routing:
- net GND: track 78.7 -> 74.2 mm
- net ANT_VCC: track 0.00 -> 3.04 mm
- net VCC_RF: track 0.00 -> 2.86 mm
- added copper zone on layer 1, net GND
- added copper zone on layer 16, net GND
Changed lines of the file:
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@@
 <layers>
 <layer number="1" name="Top" color="4" fill="1" visible="yes" active="yes"/>
-<layer number="16" name="Bottom" color="1" fill="1" visible="yes" active="yes"/>
+<layer number="16" name="Bottom" color="1" fill="1" visible="no" active="yes"/>
 <layer number="17" name="Pads" color="2" fill="1" visible="yes" active="yes"/>
 <layer number="18" name="Vias" color="2" fill="1" visible="yes" active="yes"/>
@@
 <attribute name="MF" value="Molex" x="35.56" y="-0.381" size="1.016" layer="27" font="vector" ratio="15" rot="R180" display="off"/>
 <attribute name="MPN" value="0734120110" x="35.56" y="-0.381" size="1.016" layer="27" font="vector" ratio="15" rot="R180" display="off"/>
-<attribute name="NAME" x="29.083" y="9.652" size="0.6096" layer="25" font="vector" ratio="20"/>
+<attribute name="NAME" x="31.623" y="4.572" size="0.6096" layer="25" font="vector" ratio="20"/>
 <attribute name="PROD_ID" value="CONN-09193" x="35.56" y="-0.381" size="1.016" layer="27" font="vector" ratio="15" rot="R180" display="off"/>
 <attribute name="SF_ID" value="WRL-09144" x="35.56" y="-0.381" size="1.016" layer="27" font="vector" ratio="15" rot="R180" display="off"/>
@@
 <attribute name="MF" value="Murata" x="29.21" y="12.7" size="1.016" layer="27" font="vector" ratio="15" rot="R180" display="off"/>
 <attribute name="MPN" value="BLM15HD102SN1D" x="29.21" y="12.7" size="1.016" layer="27" font="vector" ratio="15" rot="R180" display="off"/>
-<attribute name="NAME" x="29.21" y="11.684" size="0.6096" layer="25" font="vector" ratio="15" rot="R180" align="center"/>
+<attribute name="NAME" x="31.623" y="12.7" size="0.6096" layer="25" font="vector" ratio="15" align="center"/>
 <attribute name="VALUE" x="29.21" y="14.097" size="0.6096" layer="27" font="vector" ratio="15" rot="R180" align="center"/>
 </element>
@@
 <attribute name="MF" value="Murata" x="29.21" y="13.843" size="1.016" layer="27" font="vector" ratio="15" rot="R180" display="off"/>
 <attribute name="MPN" value="BLM15HD102SN1D" x="29.21" y="13.843" size="1.016" layer="27" font="vector" ratio="15" rot="R180" display="off"/>
-<attribute name="NAME" x="29.21" y="14.859" size="0.6096" layer="25" font="vector" ratio="15" rot="R180" align="center"/>
+<attribute name="NAME" x="31.623" y="13.843" size="0.6096" layer="25" font="vector" ratio="15" rot="R180" align="center"/>
 <attribute name="VALUE" x="29.21" y="15.24" size="0.6096" layer="27" font="vector" ratio="15" rot="R180" align="center"/>
 </element>
@@
 <attribute name="MPN" value="DNP" x="30.48" y="21.082" size="1.778" layer="27" display="off"/>
 </element>
+<element name="C26" library="bschulz_passives" package="C0402" value="47pF" x="30.48" y="10.033" smashed="yes">
+<attribute name="DIGIKEY" value="" x="25.4" y="20.193" size="1.778" layer="27" font="vector" display="off"/>
+<attribute name="MF" value="" x="25.4" y="20.193" size="1.778" layer="27" font="vector" display="off"/>
+<attribute name="MPN" value="" x="25.4" y="20.193" size="1.778" layer="27" font="vector" display="off"/>
+<attribute name="NAME" x="32.385" y="10.033" size="0.6096" layer="25" font="vector" ratio="15" rot="R90" align="center"/>
+<attribute name="VALUE" x="30.48" y="8.636" size="0.6096" layer="27" font="vector" ratio="15" align="center"/>
+</element>
+<element name="R28" library="bschulz_passives" package="R0402" value="10" x="29.21" y="11.176" smashed="yes" rot="R180">
+<attribute name="DIGIKEY" value="" x="38.1" y="6.096" size="1.778" layer="27" font="vector" rot="R180" display="off"/>
+<attribute name="MF" value="Yageo" x="38.1" y="6.096" size="1.778" layer="27" font="vector" rot="R180" display="off"/>
+<attribute name="MPN" value="" x="38.1" y="6.096" size="1.778" layer="27" font="vector" rot="R180" display="off"/>
+<attribute name="NAME" x="31.623" y="11.176" size="0.6096" layer="25" font="vector" ratio="15" rot="R180" align="center"/>
+<attribute name="VALUE" x="29.21" y="12.573" size="0.6096" layer="27" font="vector" ratio="15" rot="R180" align="center"/>
+<attribute name="VALUE_PART" value="" x="38.1" y="6.096" size="1.778" layer="27" font="vector" rot="R180" display="off"/>
+</element>
+<element name="FB7" library="SparkFun-Coils" library_urn="urn:adsk.eagle:library:512" package="0603" package3d_urn="urn:adsk.eagle:package:37574/1" value="30Ω/1.8A" x="28.067" y="8.89" smashed="yes" rot="R90">
+<attribute name="DIGIKEY" value="445-2986-1-ND" x="19.177" y="1.27" size="1.778" layer="27" font="vector" rot="R90" display="off"/>
+<attribute name="MF" value="TDK" x="19.177" y="1.27" size="1.778" layer="27" font="vector" rot="R90" display="off"/>
+<attribute name="MPN" value="MPZ1608D300BTA00" x="19.177" y="1.27" size="1.778" layer="27" font="vector" rot="R90" display="off"/>
+<attribute name="NAME" x="28.067" y="5.207" size="0.6096" layer="25" font="vector" ratio="20" rot="R180" align="bottom-center"/>
+<attribute name="PROD_ID" value="NDUC-07859" x="19.177" y="1.27" size="1.778" layer="27" font="vector" rot="R90" display="off"/>
+<attribute name="VALUE" x="28.829" y="8.89" size="0.6096" layer="27" font="vector" ratio="20" rot="R90" align="top-center"/>
+</element>
 </elements>
 <signals>
 <signal name="VCC_RF">
+<contactref element="R28" pad="2"/>
 <contactref element="U1" pad="14"/>
+<wire x1="28.56" y1="11.176" x2="27.813" y2="11.176" width="0.254" layer="1"/>
+<wire x1="27.178" y1="10.541" x2="25.959" y2="10.541" width="0.254" layer="1"/>
+<wire x1="27.813" y1="11.176" x2="27.178" y2="10.541" width="0.254" layer="1"/>
 </signal>
 <signal name="GND">
@@
 <wire x1="21.209" y1="11.176" x2="21.209" y2="12.192" width="0.254" layer="1"/>
 <wire x1="30.48" y1="8.614" x2="30.48" y2="5.864" width="0.4064" layer="1"/>
-<wire x1="30.48" y1="8.614" x2="28.045" y2="8.614" width="0.254" layer="1"/>
-<wire x1="28.045" y1="8.614" x2="27.813" y2="8.382" width="0.254" layer="1" curve="90"/>
-<wire x1="27.813" y1="8.382" x2="27.559" y2="8.128" width="0.254" layer="1" curve="-90"/>
 <wire x1="26.172" y1="8.128" x2="25.959" y2="8.341" width="0.254" layer="1" curve="-90"/>
-<wire x1="27.559" y1="8.128" x2="26.172" y2="8.128" width="0.254" layer="1"/>
+<polygon width="0.1524" layer="1" rank="2">
+<vertex x="32.258" y="21.987"/>
+<vertex x="32.258" y="1.635" curve="-90"/>
+<vertex x="31.258" y="0.635"/>
+<vertex x="9.89" y="0.635" curve="-90"/>
+<vertex x="8.89" y="1.635"/>
+<vertex x="8.89" y="21.987" curve="-90"/>
+<vertex x="9.89" y="22.987"/>
+<vertex x="31.258" y="22.987" curve="-90"/>
+</polygon>
+<polygon width="0.1524" layer="16">
+<vertex x="32.258" y="21.987"/>
+<vertex x="32.258" y="1.635" curve="-90"/>
+<vertex x="31.258" y="0.635"/>
+<vertex x="9.89" y="0.635" curve="-90"/>
+<vertex x="8.89" y="1.635"/>
+<vertex x="8.89" y="21.987" curve="-90"/>
+<vertex x="9.89" y="22.987"/>
+<vertex x="31.258" y="22.987" curve="-90"/>
+</polygon>
+<contactref element="C26" pad="2"/>
 </signal>
 <signal name="GPS_ANT">
@@
 <wire x1="28.953" y1="7.241" x2="28.955" y2="7.239" width="0.4064" layer="1"/>
 <polygon width="0.4064" layer="1" thermals="no">
-<vertex x="25.654" y="7.747"/>
-<vertex x="27.94" y="7.747" curve="90"/>
-<vertex x="28.194" y="8.001" curve="-90"/>
-<vertex x="28.448" y="8.255"/>
-<vertex x="29.591" y="8.255" curve="-90"/>
-<vertex x="29.845" y="8.001"/>
-<vertex x="29.845" y="6.604" curve="-90"/>
-<vertex x="29.464" y="6.223"/>
-<vertex x="28.448" y="6.223" curve="-90"/>
-<vertex x="28.194" y="6.477"/>
-<vertex x="28.194" y="6.604" curve="90"/>
-<vertex x="28.067" y="6.731"/>
-<vertex x="25.654" y="6.731" curve="-90"/>
-<vertex x="25.527" y="6.858"/>
-<vertex x="25.527" y="7.62" curve="-90"/>
+<vertex x="25.527" y="6.342"/>
+<vertex x="25.527" y="8.136" curve="-90"/>
+<vertex x="26.027" y="8.636"/>
+<vertex x="29.345" y="8.636" curve="-90"/>
+<vertex x="29.845" y="8.136"/>
+<vertex x="29.845" y="6.342" curve="-90"/>
+<vertex x="29.345" y="5.842"/>
+<vertex x="26.027" y="5.842" curve="-90"/>
 </polygon>
+<contactref element="FB7" pad="1"/>
 </signal>
 <signal name="V_BACKUP">
@@
 <wire x1="15.0917375" y1="16.041" x2="18.4563375" y2="19.4056" width="0.254" layer="1"/>
 </signal>
+<signal name="ANT_VCC">
+<contactref element="R28" pad="1"/>
+<contactref element="C26" pad="1"/>
+<contactref element="FB7" pad="2"/>
+<wire x1="28.067" y1="9.74" x2="28.36" y2="10.033" width="0.254" layer="1"/>
+<wire x1="28.36" y1="10.033" x2="29.83" y2="10.033" width="0.254" layer="1"/>
+<wire x1="29.86" y1="11.176" x2="29.83" y2="11.146" width="0.254" layer="1"/>
+<wire x1="29.83" y1="11.146" x2="29.83" y2="10.033" width="0.254" layer="1"/>
+</signal>
 </signals>
