File: MAX-M8/MAX-M8_Breakout.sch (EAGLE design)
At the start: 18 parts, among them J1 CONN_92.54_SCREW, J2 U.FL, U1 MAX-M8W

Commit message: Updated MAX-M8 breakout with active antenna support
Parts:
- added C26: 47pF, bschulz_passives:C-EUC0402
- added FB7: 30Ω/1.8A, SparkFun-Coils:FERRITE_BEAD-0603
- added R28: 10, bschulz_passives:R-EU_R0402
Connections:
- new net ANT_VCC: C26.1, FB7.2, R28.1
- new net VCC_RF: R28.2, U1.VCC_RF
- net GND: now also C26.2
- net GPS_ANT: now also FB7.1
Changed lines of the file:
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@@
 <part name="H2" library="bschulz" deviceset="MOUNTING_HOLE" device="2_NP"/>
 <part name="H3" library="bschulz" deviceset="MOUNTING_HOLE" device="2_NP"/>
+<part name="C26" library="bschulz_passives" deviceset="C-EU" device="C0402" value="47pF"/>
+<part name="R28" library="bschulz_passives" deviceset="R-EU_" device="R0402" value="10"/>
+<part name="GND36" library="SparkFun-PowerSymbols" library_urn="urn:adsk.eagle:library:530" deviceset="GND" device=""/>
+<part name="FB7" library="SparkFun-Coils" library_urn="urn:adsk.eagle:library:512" deviceset="FERRITE_BEAD" device="-0603" package3d_urn="urn:adsk.eagle:package:37574/1" value="30Ω/1.8A">
+<attribute name="DIGIKEY" value="445-2986-1-ND"/>
+<attribute name="MF" value="TDK"/>
+<attribute name="MPN" value="MPZ1608D300BTA00"/>
+</part>
 </parts>
 <sheets>
@@
 <attribute name="VALUE" x="37.592" y="94.0562" size="1.778" layer="96"/>
 </instance>
+<instance part="C26" gate="G$1" x="96.52" y="35.56" smashed="yes">
+<attribute name="NAME" x="98.044" y="35.941" size="1.778" layer="95"/>
+<attribute name="VALUE" x="98.044" y="30.861" size="1.778" layer="96"/>
+</instance>
+<instance part="R28" gate="G$1" x="104.14" y="43.18" smashed="yes">
+<attribute name="NAME" x="102.87" y="44.6786" size="1.778" layer="95"/>
+<attribute name="VALUE" x="102.87" y="39.878" size="1.778" layer="96"/>
+</instance>
+<instance part="GND36" gate="1" x="96.52" y="27.94" smashed="yes">
+<attribute name="VALUE" x="96.52" y="27.686" size="1.778" layer="96" font="vector" align="top-center"/>
+</instance>
+<instance part="FB7" gate="G$1" x="96.52" y="50.8" smashed="yes">
+<attribute name="NAME" x="97.79" y="53.34" size="1.778" layer="95" font="vector"/>
+<attribute name="VALUE" x="97.79" y="48.26" size="1.778" layer="96" font="vector" align="top-left"/>
+<attribute name="DIGIKEY" x="96.52" y="50.8" size="1.778" layer="96" display="off"/>
+<attribute name="MF" x="96.52" y="50.8" size="1.778" layer="96" display="off"/>
+<attribute name="MPN" x="96.52" y="50.8" size="1.778" layer="96" display="off"/>
+</instance>
 </instances>
 <busses>
@@
 <label x="12.7" y="83.82" size="1.016" layer="95" xref="yes"/>
 </segment>
+<segment>
+<pinref part="C26" gate="G$1" pin="2"/>
+<pinref part="GND36" gate="1" pin="GND"/>
+</segment>
 </net>
 <net name="GPS_ANT" class="0">
@@
 <wire x1="99.06" y1="58.42" x2="96.52" y2="58.42" width="0.1524" layer="91"/>
 <label x="99.06" y="58.42" size="1.27" layer="95" xref="yes"/>
+<wire x1="96.52" y1="58.42" x2="96.52" y2="55.88" width="0.1524" layer="91"/>
+<pinref part="FB7" gate="G$1" pin="1"/>
 </segment>
 <segment>
@@
 </segment>
 </net>
+<net name="VCC_RF" class="0">
+<segment>
+<pinref part="R28" gate="G$1" pin="2"/>
+<wire x1="111.76" y1="43.18" x2="109.22" y2="43.18" width="0.1524" layer="91"/>
+<label x="111.76" y="43.18" size="1.27" layer="95" xref="yes"/>
+</segment>
+<segment>
+<pinref part="U1" gate="G$1" pin="VCC_RF"/>
+<wire x1="66.04" y1="40.64" x2="71.12" y2="40.64" width="0.1524" layer="91"/>
+<label x="71.12" y="40.64" size="1.016" layer="95" xref="yes"/>
+</segment>
+</net>
+<net name="ANT_VCC" class="0">
+<segment>
+<pinref part="R28" gate="G$1" pin="1"/>
+<wire x1="99.06" y1="43.18" x2="96.52" y2="43.18" width="0.1524" layer="91"/>
+<pinref part="C26" gate="G$1" pin="1"/>
+<wire x1="96.52" y1="43.18" x2="96.52" y2="38.1" width="0.1524" layer="91"/>
+<wire x1="96.52" y1="45.72" x2="96.52" y2="43.18" width="0.1524" layer="91"/>
+<junction x="96.52" y="43.18"/>
+<pinref part="FB7" gate="G$1" pin="2"/>
+</segment>
+</net>
