File: SDI12_Interface/SDI12_Interface.brd (EAGLE design)
At the start: 34.3 x 16.1 mm, 20 parts, among them J1 CONN_6SCREW_2.54, J2 CONN_32.54_SCREW, U1 SN74LVC1G00SC70, U2 SN74LVC2G241DCU, U3 SN74LVC1G17DCK, U4 MIC5205, U5 LMR62014SOT23

Commit message: Updated part info for SDI12_Interface
Parts:
- C1, C2: value (none) -> 1uF
- C3: value (none) -> 0.1uF
- U4: value MIC5205 -> MIC5205_5V
Changed lines of the file:
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@@
 </element>
 <element name="U2" library="bschulz" package="DCU_(R-PDSO-G8)" value="SN74LVC2G241DCU" x="10.795" y="3.683" smashed="yes" rot="R270">
+<attribute name="DIGIKEY" value="296-32323-1-ND" x="10.795" y="3.683" size="1.778" layer="27" rot="R270" display="off"/>
+<attribute name="MF" value="TI" x="10.795" y="3.683" size="1.778" layer="27" rot="R270" display="off"/>
+<attribute name="MPN" value="SN74LVC2G241DCUT" x="10.795" y="3.683" size="1.778" layer="27" rot="R270" display="off"/>
 <attribute name="NAME" x="13.736" y="2.826" size="0.6096" layer="25" font="vector" ratio="15" rot="R90"/>
 <attribute name="VALUE" x="8.795" y="1.818" size="0.6096" layer="27" font="vector" ratio="15"/>
@@
 <attribute name="VALUE" x="22.86" y="10.414" size="0.6096" layer="27" font="vector" ratio="15" rot="R180" align="center"/>
 </element>
-<element name="U4" library="bschulz" package="SOT23-5" value="MIC5205" x="27.305" y="4.826" smashed="yes" rot="R90">
-<attribute name="DIGIKEY" value="" x="27.305" y="4.826" size="0.8128" layer="27" font="vector" ratio="15" rot="R90" display="off"/>
-<attribute name="MF" value="" x="27.305" y="4.826" size="0.8128" layer="27" font="vector" ratio="15" rot="R90" display="off"/>
-<attribute name="MPN" value="" x="27.305" y="4.826" size="0.8128" layer="27" font="vector" ratio="15" rot="R90" display="off"/>
+<element name="U4" library="bschulz" package="SOT23-5" value="MIC5205_5V" x="27.305" y="4.826" smashed="yes" rot="R90">
+<attribute name="DIGIKEY" value="576-1261-1-ND" x="27.305" y="4.826" size="0.8128" layer="27" font="vector" ratio="15" rot="R90" display="off"/>
+<attribute name="MF" value="Microchip" x="27.305" y="4.826" size="0.8128" layer="27" font="vector" ratio="15" rot="R90" display="off"/>
+<attribute name="MPN" value="MIC5205-5.0YM5-TR" x="27.305" y="4.826" size="0.8128" layer="27" font="vector" ratio="15" rot="R90" display="off"/>
 <attribute name="NAME" x="27.305" y="6.731" size="0.6096" layer="25" font="vector" ratio="15" rot="R180" align="center"/>
 <attribute name="VALUE" x="27.178" y="7.112" size="0.6096" layer="27" font="vector" ratio="15" rot="R180" align="center"/>
 </element>
-<element name="C1" library="bschulz_passives" package="C0603" value="" x="27.305" y="2.159" smashed="yes" rot="R180">
+<element name="C1" library="bschulz_passives" package="C0603" value="1uF" x="27.305" y="2.159" smashed="yes" rot="R180">
 <attribute name="DIGIKEY" value="587-1251-1-ND" x="27.305" y="2.159" size="0.8128" layer="27" font="vector" ratio="15" rot="R180" display="off"/>
 <attribute name="MF" value="Yaiyo Yuden" x="27.305" y="2.159" size="0.8128" layer="27" font="vector" ratio="15" rot="R180" display="off"/>
@@
 <attribute name="VALUE" x="27.305" y="3.556" size="0.6096" layer="27" font="vector" ratio="15" rot="R180" align="center"/>
 </element>
-<element name="C2" library="bschulz_passives" package="C0603" value="" x="24.003" y="4.826" smashed="yes" rot="R90">
+<element name="C2" library="bschulz_passives" package="C0603" value="1uF" x="24.003" y="4.826" smashed="yes" rot="R90">
 <attribute name="DIGIKEY" value="587-1251-1-ND" x="24.003" y="4.826" size="0.8128" layer="27" font="vector" ratio="15" rot="R90" display="off"/>
 <attribute name="MF" value="Yaiyo Yuden" x="24.003" y="4.826" size="0.8128" layer="27" font="vector" ratio="15" rot="R90" display="off"/>
@@
 <attribute name="VALUE" x="25.4" y="4.826" size="0.6096" layer="27" font="vector" ratio="15" rot="R90" align="center"/>
 </element>
-<element name="C3" library="bschulz_passives" package="C0603" value="" x="10.287" y="8.509" smashed="yes">
+<element name="C3" library="bschulz_passives" package="C0603" value="0.1uF" x="10.287" y="8.509" smashed="yes">
 <attribute name="DIGIKEY" value="490-6051-1-ND" x="10.287" y="8.509" size="0.8128" layer="27" font="vector" ratio="15" display="off"/>
 <attribute name="MF" value="Murata" x="10.287" y="8.509" size="0.8128" layer="27" font="vector" ratio="15" display="off"/>
@@
 <via x="27.305" y="4.826" extent="1-16" drill="0.35"/>
 <wire x1="27.305" y1="4.826" x2="27.305" y2="11.684" width="0.3048" layer="16"/>
+<wire x1="20.828" y1="11.684" x2="21.91" y2="11.303" width="0" layer="19" extent="1-1"/>
+<wire x1="20.828" y1="10.795" x2="20.828" y2="11.684" width="0" layer="19" extent="1-1"/>
+<wire x1="19.842" y1="10.287" x2="20.828" y2="10.795" width="0" layer="19" extent="1-1"/>
+<wire x1="18.542" y1="10.287" x2="19.842" y2="10.287" width="0" layer="19" extent="1-1"/>
+<wire x1="18.095" y1="7.493" x2="18.542" y2="10.287" width="0" layer="19" extent="1-1"/>
 </signal>
 <signal name="VIN">
@@
 <wire x1="9.437" y1="8.509" x2="9.437" y2="9.564" width="0.254" layer="1"/>
 <wire x1="9.437" y1="9.564" x2="9.525" y2="9.652" width="0.254" layer="1"/>
+<wire x1="15.494" y1="9.31" x2="17.242" y2="9.337" width="0" layer="19" extent="1-1"/>
+<wire x1="16.195" y1="7.493" x2="15.494" y2="9.31" width="0" layer="19" extent="1-1"/>
+<wire x1="17.694" y1="5.08" x2="16.195" y2="7.493" width="0" layer="19" extent="1-1"/>
 </signal>
 <signal name="TX">
@@
 <vertex x="19.177" y="9.652"/>
 </polygon>
+<wire x1="19.842" y1="9.337" x2="21.185" y2="9.144" width="0" layer="19" extent="1-1"/>
+<wire x1="19.644" y1="5.08" x2="19.842" y2="9.337" width="0" layer="19" extent="1-1"/>
 </signal>
 <signal name="5V">

Commit message: Fixed inverter in SDI-12 interface
SDI-12 interface erroneously had non-inverting buffer instead of inverting buffer
Parts:
- U3: value SN74LVC1G17DCK -> (none)
Changed lines of the file:
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@@
 <layer number="56" name="wert" color="7" fill="1" visible="no" active="no"/>
 <layer number="57" name="tCAD" color="7" fill="1" visible="no" active="no"/>
+<layer number="58" name="bCAD" color="7" fill="1" visible="no" active="no"/>
 <layer number="59" name="tCarbon" color="7" fill="1" visible="no" active="no"/>
 <layer number="60" name="bCarbon" color="7" fill="1" visible="no" active="no"/>
@@
 <layer number="128" name="_bValues" color="7" fill="1" visible="no" active="yes"/>
 <layer number="129" name="Mask" color="7" fill="1" visible="no" active="yes"/>
+<layer number="130" name="SMDSTROOK" color="7" fill="1" visible="no" active="no"/>
 <layer number="131" name="tAdjust" color="7" fill="1" visible="no" active="yes"/>
 <layer number="132" name="bAdjust" color="7" fill="1" visible="no" active="yes"/>
+<layer number="133" name="bottom_silk" color="7" fill="1" visible="no" active="no"/>
+<layer number="134" name="mbFinish" color="7" fill="1" visible="no" active="no"/>
+<layer number="135" name="mtGlue" color="7" fill="1" visible="no" active="no"/>
+<layer number="136" name="mbGlue" color="7" fill="1" visible="no" active="no"/>
+<layer number="137" name="mtTest" color="7" fill="1" visible="no" active="no"/>
+<layer number="138" name="mbTest" color="7" fill="1" visible="no" active="no"/>
+<layer number="139" name="mtKeepout" color="7" fill="1" visible="no" active="no"/>
+<layer number="140" name="mbKeepout" color="7" fill="1" visible="no" active="no"/>
+<layer number="141" name="mtRestrict" color="7" fill="1" visible="no" active="no"/>
+<layer number="142" name="mbRestrict" color="7" fill="1" visible="no" active="no"/>
+<layer number="143" name="mvRestrict" color="7" fill="1" visible="no" active="no"/>
 <layer number="144" name="Drill_legend" color="7" fill="1" visible="no" active="yes"/>
+<layer number="145" name="mHoles" color="7" fill="1" visible="no" active="no"/>
+<layer number="146" name="mMilling" color="7" fill="1" visible="no" active="no"/>
+<layer number="147" name="mMeasures" color="7" fill="1" visible="no" active="no"/>
+<layer number="148" name="mDocument" color="7" fill="1" visible="no" active="no"/>
+<layer number="149" name="mReference" color="7" fill="1" visible="no" active="no"/>
 <layer number="150" name="Notes" color="7" fill="1" visible="no" active="yes"/>
 <layer number="151" name="HeatSink" color="7" fill="1" visible="no" active="yes"/>
@@
 <layer number="154" name="FabDoc2" color="7" fill="1" visible="no" active="yes"/>
 <layer number="155" name="FabDoc3" color="7" fill="1" visible="no" active="yes"/>
+<layer number="166" name="AntennaArea" color="7" fill="1" visible="no" active="no"/>
+<layer number="168" name="4mmHeightArea" color="7" fill="1" visible="no" active="no"/>
+<layer number="191" name="mNets" color="7" fill="1" visible="no" active="no"/>
+<layer number="192" name="mBusses" color="7" fill="1" visible="no" active="no"/>
+<layer number="193" name="mPins" color="7" fill="1" visible="no" active="no"/>
+<layer number="194" name="mSymbols" color="7" fill="1" visible="no" active="no"/>
+<layer number="195" name="mNames" color="7" fill="1" visible="no" active="no"/>
+<layer number="196" name="mValues" color="7" fill="1" visible="no" active="no"/>
 <layer number="199" name="Contour" color="7" fill="1" visible="no" active="yes"/>
 <layer number="200" name="200bmp" color="7" fill="1" visible="no" active="yes"/>
@@
 <attribute name="VALUE" x="8.795" y="1.818" size="0.6096" layer="27" font="vector" ratio="15"/>
 </element>
-<element name="U3" library="bschulz" package="DCK_R-PDSO-G5" value="SN74LVC1G17DCK" x="10.287" y="6.096" smashed="yes" rot="R90">
-<attribute name="DIGIKEY" value="296-11934-1-ND" x="24.257" y="31.496" size="1.778" layer="27" rot="R90" display="off"/>
-<attribute name="DISP" value="SN74LVC1G17" x="24.257" y="31.496" size="1.778" layer="27" rot="R90" display="off"/>
+<element name="U3" library="bschulz" package="DCK_R-PDSO-G5" value="" x="10.287" y="6.096" smashed="yes" rot="R90">
+<attribute name="DIGIKEY" value="296-11608-1-ND" x="24.257" y="31.496" size="1.778" layer="27" rot="R90" display="off"/>
+<attribute name="DISP" value="SN74LVC1G14" x="24.257" y="31.496" size="1.778" layer="27" rot="R90" display="off"/>
 <attribute name="MF" value="TI" x="24.257" y="31.496" size="1.778" layer="27" rot="R90" display="off"/>
-<attribute name="MPN" value="SN74LVC1G17DCKR" x="24.257" y="31.496" size="1.778" layer="27" rot="R90" display="off"/>
+<attribute name="MPN" value="SN74LVC1G14DCKR" x="24.257" y="31.496" size="1.778" layer="27" rot="R90" display="off"/>
 <attribute name="NAME" x="12.192" y="6.477" size="0.6096" layer="25" font="vector" ratio="15" rot="R270" align="center"/>
 <attribute name="VALUE" x="10.287" y="7.62" size="0.6096" layer="27" font="vector" ratio="15" rot="R180" align="center"/>

Commit message: Backlog of various boards
Parts:
- U3: value (none) -> SN74LVC1G17DCK
Changed lines of the file:
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@@
 <layer number="56" name="wert" color="7" fill="1" visible="no" active="no"/>
 <layer number="57" name="tCAD" color="7" fill="1" visible="no" active="no"/>
-<layer number="58" name="bCAD" color="7" fill="1" visible="no" active="no"/>
 <layer number="59" name="tCarbon" color="7" fill="1" visible="no" active="no"/>
 <layer number="60" name="bCarbon" color="7" fill="1" visible="no" active="no"/>
@@
 <layer number="128" name="_bValues" color="7" fill="1" visible="no" active="yes"/>
 <layer number="129" name="Mask" color="7" fill="1" visible="no" active="yes"/>
-<layer number="130" name="SMDSTROOK" color="7" fill="1" visible="no" active="no"/>
 <layer number="131" name="tAdjust" color="7" fill="1" visible="no" active="yes"/>
 <layer number="132" name="bAdjust" color="7" fill="1" visible="no" active="yes"/>
-<layer number="133" name="bottom_silk" color="7" fill="1" visible="no" active="no"/>
-<layer number="134" name="mbFinish" color="7" fill="1" visible="no" active="no"/>
-<layer number="135" name="mtGlue" color="7" fill="1" visible="no" active="no"/>
-<layer number="136" name="mbGlue" color="7" fill="1" visible="no" active="no"/>
-<layer number="137" name="mtTest" color="7" fill="1" visible="no" active="no"/>
-<layer number="138" name="mbTest" color="7" fill="1" visible="no" active="no"/>
-<layer number="139" name="mtKeepout" color="7" fill="1" visible="no" active="no"/>
-<layer number="140" name="mbKeepout" color="7" fill="1" visible="no" active="no"/>
-<layer number="141" name="mtRestrict" color="7" fill="1" visible="no" active="no"/>
-<layer number="142" name="mbRestrict" color="7" fill="1" visible="no" active="no"/>
-<layer number="143" name="mvRestrict" color="7" fill="1" visible="no" active="no"/>
 <layer number="144" name="Drill_legend" color="7" fill="1" visible="no" active="yes"/>
-<layer number="145" name="mHoles" color="7" fill="1" visible="no" active="no"/>
-<layer number="146" name="mMilling" color="7" fill="1" visible="no" active="no"/>
-<layer number="147" name="mMeasures" color="7" fill="1" visible="no" active="no"/>
-<layer number="148" name="mDocument" color="7" fill="1" visible="no" active="no"/>
-<layer number="149" name="mReference" color="7" fill="1" visible="no" active="no"/>
 <layer number="150" name="Notes" color="7" fill="1" visible="no" active="yes"/>
 <layer number="151" name="HeatSink" color="7" fill="1" visible="no" active="yes"/>
@@
 <layer number="154" name="FabDoc2" color="7" fill="1" visible="no" active="yes"/>
 <layer number="155" name="FabDoc3" color="7" fill="1" visible="no" active="yes"/>
-<layer number="166" name="AntennaArea" color="7" fill="1" visible="no" active="no"/>
-<layer number="168" name="4mmHeightArea" color="7" fill="1" visible="no" active="no"/>
-<layer number="191" name="mNets" color="7" fill="1" visible="no" active="no"/>
-<layer number="192" name="mBusses" color="7" fill="1" visible="no" active="no"/>
-<layer number="193" name="mPins" color="7" fill="1" visible="no" active="no"/>
-<layer number="194" name="mSymbols" color="7" fill="1" visible="no" active="no"/>
-<layer number="195" name="mNames" color="7" fill="1" visible="no" active="no"/>
-<layer number="196" name="mValues" color="7" fill="1" visible="no" active="no"/>
 <layer number="199" name="Contour" color="7" fill="1" visible="no" active="yes"/>
 <layer number="200" name="200bmp" color="7" fill="1" visible="no" active="yes"/>
@@
 <attribute name="VALUE" x="8.795" y="1.818" size="0.6096" layer="27" font="vector" ratio="15"/>
 </element>
-<element name="U3" library="bschulz" package="DCK_R-PDSO-G5" value="" x="10.287" y="6.096" smashed="yes" rot="R90">
-<attribute name="DIGIKEY" value="296-11608-1-ND" x="24.257" y="31.496" size="1.778" layer="27" rot="R90" display="off"/>
-<attribute name="DISP" value="SN74LVC1G14" x="24.257" y="31.496" size="1.778" layer="27" rot="R90" display="off"/>
+<element name="U3" library="bschulz" package="DCK_R-PDSO-G5" value="SN74LVC1G17DCK" x="10.287" y="6.096" smashed="yes" rot="R90">
+<attribute name="DIGIKEY" value="296-11934-1-ND" x="24.257" y="31.496" size="1.778" layer="27" rot="R90" display="off"/>
+<attribute name="DISP" value="SN74LVC1G17" x="24.257" y="31.496" size="1.778" layer="27" rot="R90" display="off"/>
 <attribute name="MF" value="TI" x="24.257" y="31.496" size="1.778" layer="27" rot="R90" display="off"/>
-<attribute name="MPN" value="SN74LVC1G14DCKR" x="24.257" y="31.496" size="1.778" layer="27" rot="R90" display="off"/>
+<attribute name="MPN" value="SN74LVC1G17DCKR" x="24.257" y="31.496" size="1.778" layer="27" rot="R90" display="off"/>
 <attribute name="NAME" x="12.192" y="6.477" size="0.6096" layer="25" font="vector" ratio="15" rot="R270" align="center"/>
 <attribute name="VALUE" x="10.287" y="7.62" size="0.6096" layer="27" font="vector" ratio="15" rot="R180" align="center"/>
